File: hardware/reflowoven.sch (KiCad schematic (older format))
At the start: 11 parts

Commit message: fix value miss
Parts:
- R? (x2): value 4.7K -> 1.5k; symbol R -> R-RESCUE-reflowoven
- R? (x2): value 2.2K -> 3.3k; symbol R -> R-RESCUE-reflowoven
Changed lines of the file:
@@
 EESchema Schematic File Version 2
+LIBS:reflowoven-rescue
 LIBS:power
 LIBS:device
@@
 LIBS:memory
 LIBS:xilinx
-LIBS:special
 LIBS:microcontrollers
 LIBS:dsp
@@
 LIBS:contrib
 LIBS:valves
+LIBS:reflowoven-cache
 EELAYER 25 0
 EELAYER END
@@
 Connection ~ 4019 4992
 $Comp
-L GND #PWR?
+L GND-RESCUE-reflowoven #PWR?
 U 1 1 554F68F1
 P 4019 5337
@@
 Connection ~ 7511 5841
 $Comp
-L GND #PWR?
+L GND-RESCUE-reflowoven #PWR?
 U 1 1 554F6F9E
 P 7511 6137
@@
 SSR
 $Comp
-L R R?
+L R-RESCUE-reflowoven R?
 U 1 1 554F77EE
 P 7570 1925
 F 0 "R?" V 7650 1925 40  0000 C CNN
-F 1 "4.7K" V 7577 1926 40  0000 C CNN
+F 1 "1.5k" V 7577 1926 40  0000 C CNN
 F 2 "" V 7500 1925 30  0000 C CNN
 F 3 "" H 7570 1925 30  0000 C CNN
@@
 $EndComp
 $Comp
-L R R?
+L R-RESCUE-reflowoven R?
 U 1 1 554F78A1
 P 7570 2519
 F 0 "R?" V 7650 2519 40  0000 C CNN
-F 1 "2.2K" V 7577 2520 40  0000 C CNN
+F 1 "3.3k" V 7577 2520 40  0000 C CNN
 F 2 "" V 7500 2519 30  0000 C CNN
 F 3 "" H 7570 2519 30  0000 C CNN
@@
 $EndComp
 $Comp
-L GND #PWR?
+L GND-RESCUE-reflowoven #PWR?
 U 1 1 554F79C5
 P 8520 2900
@@
 	7570 2175 7570 2269
 $Comp
-L R R?
+L R-RESCUE-reflowoven R?
 U 1 1 554F92CD
 P 7797 3203
 F 0 "R?" V 7877 3203 40  0000 C CNN
-F 1 "4.7K" V 7804 3204 40  0000 C CNN
+F 1 "1.5k" V 7804 3204 40  0000 C CNN
 F 2 "" V 7727 3203 30  0000 C CNN
 F 3 "" H 7797 3203 30  0000 C CNN
@@
 $EndComp
 $Comp
-L R R?
+L R-RESCUE-reflowoven R?
 U 1 1 554F92D3
 P 7797 3797
 F 0 "R?" V 7877 3797 40  0000 C CNN
-F 1 "2.2K" V 7804 3798 40  0000 C CNN
+F 1 "3.3k" V 7804 3798 40  0000 C CNN
 F 2 "" V 7727 3797 30  0000 C CNN
 F 3 "" H 7797 3797 30  0000 C CNN
@@
 	7570 2769 7570 2882
 $Comp
-L GND #PWR?
+L GND-RESCUE-reflowoven #PWR?
 U 1 1 554F9FE1
 P 7570 2882
@@
 	7797 4047 7797 4129
 $Comp
-L GND #PWR?
+L GND-RESCUE-reflowoven #PWR?
 U 1 1 554FA11F
 P 7797 4129
